Commit message: revised height and angle of the camera for better image capturing

File: mir_robot/mir_description/urdf/mir.urdf.xacro (robot description, xacro)
@@ -7,5 +7,5 @@
   <xacro:include filename="$(find mir_description)/urdf/include/_d435.urdf.xacro" />
   <xacro:sensor_d435 parent="base_link" name="camera">
-    <origin xyz="0 0 0.60" rpy="0 0 0"/>
+    <origin xyz="0 0 1.70" rpy="0 0.087 0"/>
   </xacro:sensor_d435>
   <xacro:arg name="tf_prefix" default="" />
